File: hps_clock/hps_clock.kicad_sch (KiCad schematic)
At the start: 4 parts

Commit message: mcu schematic
Parts:
- added C4, C5: C_0805_22pf, footprints:C_0805_2012Metric, symbol HPS:C_0805_22pf
- added C? (x2): C_0805_0.1uf, footprints:C_0805_2012Metric, symbol HPS:C_0805_0.1uf
- added R3: R_0805_10K, footprints:R_0805_2012Metric, symbol HPS:R_0805_10K
- added U1: ATmega328-PU, footprints:DIP-28_W7.62mm, symbol HPS:ATmega328-PU
- added Y1: Crystal_16MHz, footprints:Crystal_SMD_HC49-SD, symbol HPS:Crystal_16MHz
Connections:
- new net: C5.2, U1.10 (XTAL2/PB7), Y1.2
- new net: C?.1, U1.21 (AREF)
- new net: C4.2, U1.9 (XTAL1/PB6), Y1.1
- new net GND: C4.1, C5.1, C?.2, C?.2, U1.22 (GND), U1.8 (GND)
- new net LED_SCK: U1.19 (PB5)
- new net RESEST: R3.2, U1.1 (~{RESET}/PC6)
- new net RXD: U1.2 (PD0)
- new net TXD: U1.3 (PD1)
- new net VCC: C?.1, R3.1, U1.20 (AVCC), U1.7 (VCC)
