File: hps_clock/hps_clock.kicad_sch (KiCad schematic)
At the start: 11 parts, among them U1 ATmega328-PU, Y1 Crystal_16MHz

Commit message: schematic w2
Parts:
- added C3, C9: C_0805_0.1uf, footprints:C_0805_2012Metric, symbol HPS:C_0805_0.1uf
- added C8: C_0805_1uf, footprints:C_0805_2012Metric, symbol HPS:C_0805_1uf
- added D1: LED_0805, footprints:LED_0805_2012Metric, symbol HPS:LED_0805
- added J1: Conn_01x06, footprints:PinHeader_1x06_P2.54mm_Vertical, symbol HPS:Conn_01x06
- added J3: Barrel_Jack_Switch, footprints:PJ-102AH, symbol HPS:Barrel_Jack_Switch
- added R1: R_0805_2.2K, footprints:R_0805_2012Metric, symbol HPS:R_0805_2.2K
- added R4, R5: R_0805_47, footprints:R_0805_2012Metric, symbol HPS:R_0805_47
- added SW1: Omron_B3F_SPST, footprints:SW_SPST_Omron_B3FS-100xP, symbol HPS:Omron_B3F_SPST
- added U4: L7805, symbol HPS:L7805
Connections:
- net GND: now also C8.2, C9.2, J1.1 (Pin_1), J1.2 (Pin_2), J3.2, R1.2, SW1.1 (A), SW1.2 (A), U4.2 (GND)
- net LED_SCK: now also D1.2 (A)
- net RXD: now also R4.1
- net TXD: now also R5.1
- net VCC: now also C9.1, U4.3 (OUT)
- new net: D1.1 (K), R1.1
- new net: J1.4 (Pin_4), R5.2
- new net: J1.5 (Pin_5), R4.2
- new net: C3.2, J1.6 (Pin_6)
- new net: C8.1, J3.1, U4.1 (IN)
- new net RESET: C3.1, SW1.3 (B), SW1.4 (B)
- no-connect marks 0 -> 2

Commit message: schematic w2 v2.1
Parts:
- J3: symbol HPS:Barrel_Jack_Switch -> HPS:PJ-102AH; Digikey PN (none) -> CP-102AH-ND; MFG (none) -> CUI Devices; MPN (none) -> PJ-102AH; Mouser PN (none) -> 490-PJ-102AH
- gave numbers to parts that had none: 2
Other:
- note added: "LED"
- note added: "MCU"
- note added: "Power Input"
- note added: "Serial"

Commit message: schematic w2 v2.2
Connections:
- net RESET renamed ~{RESET}
Changed lines of the file:
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@@
     )
   )
-  (global_label "RESET" (shape output) (at 35.56 72.39 180) (fields_autoplaced)
+  (global_label "~{RESET}" (shape output) (at 35.56 72.39 180) (fields_autoplaced)
     (effects (font (size 1.27 1.27)) (justify right))
     (property "Intersheet References" "${INTERSHEET_REFS}" (id 0) (at 27.4017 72.3106 0)

Commit message: schematic w2 v2.3
Connections:
- net RESEST renamed RESET
Changed lines of the file:
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@@
     )
   )
-  (global_label "RESEST" (shape input) (at 222.25 118.11 0) (fields_autoplaced)
+  (global_label "RESET" (shape input) (at 222.25 118.11 0) (fields_autoplaced)
     (effects (font (size 1.27 1.27)) (justify left))
-    (property "Intersheet References" "${INTERSHEET_REFS}" (id 0) (at 231.6179 118.0306 0)
+    (property "Intersheet References" "${INTERSHEET_REFS}" (id 0) (at 230.4083 118.0306 0)
       (effects (font (size 1.27 1.27)) (justify left) hide)
     )

Commit message: schematic w2 v2.4
Connections:
- net RESET is gone; now on net ~{RESET}: R3.2, U1.1 (~{RESET}/PC6)
Changed lines of the file:
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@@
     )
   )
-  (global_label "RESET" (shape input) (at 222.25 118.11 0) (fields_autoplaced)
+  (global_label "~{RESET}" (shape input) (at 222.25 118.11 0) (fields_autoplaced)
     (effects (font (size 1.27 1.27)) (justify left))
     (property "Intersheet References" "${INTERSHEET_REFS}" (id 0) (at 230.4083 118.0306 0)

Commit message: week3
Parts:
- added BT?: Battery_Cell, footprints:BatteryHolder_Keystone_106_1x20mm, symbol HPS:Battery_Cell
- added R1: PhotoconductivePhotocell, footprints:R_LDR_4.9x4.2mm_P2.54mm_Vertical, symbol HPS:PhotoconductivePhotocell
- added R10, R9: R_0805_4.7K, footprints:R_0805_2012Metric, symbol HPS:R_0805_4.7K
- added R11: R_0805_100K, footprints:R_0805_2012Metric, symbol HPS:R_0805_100K
- added R6, R7, R8: R_0805_10K, footprints:R_0805_2012Metric, symbol HPS:R_0805_10K
- added SW2, SW3, SW4: Omron_B3F_SPST, footprints:SW_SPST_Omron_B3FS-100xP, symbol HPS:Omron_B3F_SPST
- added U1: DS1307_DIP-8, footprints:DIP-8_W7.62mm, symbol HPS:DS1307_DIP-8
Connections:
- net GND: now also BT?.2 (-), R11.2, SW2.1 (A), SW2.2 (A), SW3.1 (A), SW3.2 (A), SW4.1 (A), SW4.2 (A), U1.4 (GND)
- net VCC: now also R1.1, R10.1, R6.1, R7.1, R8.1, R9.1, U1.8 (VCC)
- net LIGHT_SENSOR: now reaches U1.23 (PC0)
- net LIGHT_SENSOR: now also R1.2, R11.1
- net SDA: now reaches U1.27 (PC4)
- net SDA: now also R9.2, U1.5 (SDA)
- net SCL: now reaches U1.28 (PC5)
- net SCL: now also R10.2, U1.6 (SCL)
- net UP: now reaches U1.4 (PD2)
- net UP: now also R6.2, SW2.3 (B), SW2.4 (B)
- net DOWN: now reaches U1.5 (PD3)
- net DOWN: now also R7.2, SW3.3 (B), SW3.4 (B)
- net MULTI: now reaches U1.6 (PD4)
- net MULTI: now also R8.2, SW4.3 (B), SW4.4 (B)
- new net: BT?.1 (+), U1.3 (VBAT)
- no-connect marks 2 -> 3
Other:
- note added: "LIGHT_SENSOR"
- note added: "Real Time Clock"
- moved on the sheet: D1, R1

Commit message: week3/4
Parts:
- removed R8: R_0805_10K, footprints:R_0805_2012Metric, symbol HPS:R_0805_10K
- added R6: R_0805_10K, footprints:R_0805_2012Metric, symbol HPS:R_0805_10K
- gave numbers to parts that had none: 1
- renumbered C3 to C1, C8 to C2, C9 to C3, C1 to C4, C2 to C5, C4 to C6, C5 to C7, J3 to J1, J1 to J2, R3 to R10, R1 to R11, R11 to R2, R4 to R3, R5 to R4, R6 to R5, R9 to R8, R10 to R9, U4 to U2, U1 to U3
Connections:
- net DOWN: now also SW3.1 (A), SW3.2 (A), R6.1; no longer R7.2, SW3.3 (B), SW3.4 (B)
- net GND: now also R5.2, R7.2, R6.2; no longer SW2.1 (A), SW2.2 (A), SW3.1 (A), SW3.2 (A), SW4.1 (A), SW4.2 (A)
- net MULTI: now also R7.1, SW4.1 (A), SW4.2 (A); no longer SW4.3 (B), SW4.4 (B)
- net UP: now also R5.1, SW2.1 (A), SW2.2 (A); no longer R5.2, SW2.3 (B), SW2.4 (B)
- net VCC: now also SW2.3 (B), SW2.4 (B), SW3.3 (B), SW3.4 (B), SW4.3 (B), SW4.4 (B); no longer R5.1, R7.1
Other:
- moved on the sheet: R10, R5, R8, R9, SW2

Commit message: schematic done..?
Parts:
- added C8: C_0805_0.1uf, footprints:C_0805_2012Metric, symbol HPS:C_0805_0.1uf
- added C9: C_0805_10uf, footprints:C_0805_2012Metric, symbol HPS:C_0805_10uf
- added DS1: LED_Display_1001, footprints:Adafruit-1001-0-0-MFG, symbol HPS:LED_Display_1001
- added R12: R_0805_22K, footprints:R_0805_2012Metric, symbol HPS:R_0805_22K
- added U4: MAX7219, footprints:DIP-24_W7.62mm, symbol HPS:MAX7219
- U2: footprint (none) -> footprints:TO-252-2
- renumbered R9 to R10, R10 to R11, R11 to R5, R5 to R6, R6 to R7, R7 to R8, R8 to R9
Connections:
- net GND: now also C8.2, C9.2, U4.4 (GND), U4.9 (GND)
- net VCC: now also C8.1, C9.1, R12.1, U4.19 (V+)
- net at U3.14 (PB0): now also U4.12 (LOAD)
- net at U3.15 (PB1): now also U4.13 (CLK)
- net at U3.16 (PB2): now also U4.1 (DIN)
- new net: DS1.1 (E), U4.21 (SEG_E)
- new net: DS1.10 (COM_DIG.3), U4.6 (DIG_2)
- new net: DS1.11 (COM_DIG.2), U4.11 (DIG_1)
- new net: DS1.12 (F), U4.15 (SEG_F)
- new net: DS1.13 (A), U4.14 (SEG_A)
- new net: DS1.14 (COM_DIG.1), U4.2 (DIG_0)
- new net: DS1.2 (D), U4.23 (SEG_D)
- new net: DS1.3 (DP), DS1.8 (COLON), U4.22 (SEG_DP)
- new net: DS1.4 (C), U4.20 (SEG_C)
- new net: DS1.5 (G), U4.17 (SEG_G)
- new net: DS1.6 (COM_DIG.4), U4.7 (DIG_3)
- new net: DS1.7 (COM_COLON), U4.3 (DIG_4)
- new net: DS1.9 (B), U4.16 (SEG_B)
- new net: R12.2, U4.18 (ISET)
- no-connect marks 3 -> 7
Other:
- note added: "Display Driver + Seven Segment Display"
- moved on the sheet: BT1, C1, C2, C3, C4, C5, C6, C7, D1, H1, H2, H3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
