File: hps_clock/hps_clock.kicad_sch (KiCad schematic)
At the start: 39 parts, among them J1 Barrel_Jack_Switch, J2 Conn_01x06, SW1 Omron_B3F_SPST, SW2 Omron_B3F_SPST, SW3 Omron_B3F_SPST, SW4 Omron_B3F_SPST, U1 DS1307_DIP-8, U2 L7805, U3 ATmega328-PU, U4 MAX7219, Y1 Crystal_16MHz

Commit message: schematic_fin
Parts:
- added J3: Conn_02x03_Odd_Even, footprints:PinHeader_2x03_P2.54mm_Vertical, symbol HPS:Conn_02x03_Odd_Even
- added Y1: Crystal_32768Hz, footprints:Crystal_SMD_2Pin_3.2x1.5mm, symbol HPS:Crystal_32768Hz
- renumbered R5 to R1, R1 to R2, R2 to R3, R3 to R4, R4 to R5, U2 to U1, U1 to U2, Y1 to Y2
Connections:
- net GND: now also J3.6 (Pin_6)
- net LED_SCK: now also J3.3 (Pin_3)
- net VCC: now also J3.2 (Pin_2); no longer SW2.4 (B)
- net ~{RESET}: now also J3.5 (Pin_5)
- net DISP_LOAD: now reaches U3.14 (PB0), U4.12 (LOAD)
- net DISP_CLK: now reaches U3.15 (PB1), U4.13 (CLK)
- net DISP_DATA: now reaches U3.16 (PB2), U4.1 (DIN)
- net MOSI: now reaches U3.17 (PB3)
- net MOSI: now also J3.4 (Pin_4)
- net MISO: now reaches U3.18 (PB4)
- net MISO: now also J3.1 (Pin_1)
- net at U2.1 (X1): now also Y1.1
- net at U2.2 (X2): now also Y1.2
- net DOWN renamed BTN_SEL
- net MULTI renamed BTN_UP
- net UP renamed BTN_DWN
- no-connect marks 7 -> 13
Other:
- note added: "Buttons"
- note added: "ICSP"
- note added: "Mechanical"
- moved on the sheet: BT1, C1, C2, C3, C4, C5, C6, C7, C8, C9, D1, DS1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

Commit message: schematic_final
Connections:
- net VCC: now also SW2.4 (B)
Changed lines of the file:
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@@
   (junction (at 80.01 195.58) (diameter 0) (color 0 0 0 0)
+  )
+  (junction (at 207.01 350.52) (diameter 0) (color 0 0 0 0)
   )
   (junction (at 391.16 149.86) (diameter 0) (color 0 0 0 0)
@@
     (stroke (width 0) (type default) (color 0 0 0 0))
   )
+  (wire (pts (xy 207.01 350.52) (xy 209.55 350.52))
+    (stroke (width 0) (type default) (color 0 0 0 0))
+  )

Commit message: pcb_5
Parts:
- added TP1, TP2, TP3, TP4, TP5, TP6: TestPoint, footprints:TestPoint_THTPad_D2.0mm_Drill1.0mm, symbol HPS:TestPoint
- J1: footprint footprints:PJ-102AH -> footprints:Wurth-694106402002; symbol HPS:PJ-102AH -> HPS:Power_inlet_vertical; Digikey PN CP-102AH-ND -> 732-5931-ND; MFG CUI Devices -> Wurth; MPN PJ-102AH -> 694106402002
Connections:
- net DISP_CLK is gone; now on net GND: U3.15 (PB1), U4.13 (CLK)
- net DISP_DATA is gone; now on net GND: U3.16 (PB2), U4.1 (DIN)
- net DISP_LOAD is gone; now on net GND: U3.14 (PB0), U4.12 (LOAD)
- net SCL is gone; now on net GND: R10.2, U2.6 (SCL), U3.28 (PC5)
- net SDA is gone; now on net GND: R9.2, U2.5 (SDA), U3.27 (PC4)
- net VCC is gone; now on net GND: C3.1, C5.1, C8.1, C9.1, J3.2 (Pin_2), R10.1, R11.1, R12.1, R2.1, R9.1, SW2.3 (B), SW2.4 (B), SW3.3 (B), SW3.4 (B), SW4.3 (B), SW4.4 (B), U1.3 (OUT), U2.8 (VCC), U3.20 (AVCC), U3.7 (VCC), U4.19 (V+)
- net GND: now also TP1.1, TP2.1, TP3.1, TP4.1, TP5.1, TP6.1

Commit message: pcb_6
Parts:
- added TP7, TP8: TestPoint, footprints:TestPoint_THTPad_D2.0mm_Drill1.0mm, symbol HPS:TestPoint
Connections:
- net GND: now also TP7.1, TP8.1; no longer C3.1, C5.1, C8.1, C9.1, J3.2 (Pin_2), R10.1, R10.2, R11.1, R12.1, R2.1, R9.1, R9.2, SW2.3 (B), SW2.4 (B), SW3.3 (B), SW3.4 (B), SW4.3 (B), SW4.4 (B), TP1.1, TP2.1, TP3.1, TP4.1, TP5.1, TP6.1, U1.3 (OUT), U2.5 (SDA), U2.6 (SCL), U2.8 (VCC), U3.14 (PB0), U3.15 (PB1), U3.16 (PB2), U3.20 (AVCC), U3.27 (PC4), U3.28 (PC5), U3.7 (VCC), U4.1 (DIN), U4.12 (LOAD), U4.13 (CLK), U4.19 (V+)
- new net DISP_CLK: TP6.1, U3.15 (PB1), U4.13 (CLK)
- new net DISP_DATA: TP5.1, U3.16 (PB2), U4.1 (DIN)
- new net DISP_LOAD: TP4.1, U3.14 (PB0), U4.12 (LOAD)
- new net SCL: R10.2, TP1.1, U2.6 (SCL), U3.28 (PC5)
- new net SDA: R9.2, TP2.1, U2.5 (SDA), U3.27 (PC4)
- new net VCC: C3.1, C5.1, C8.1, C9.1, J3.2 (Pin_2), R10.1, R11.1, R12.1, R2.1, R9.1, SW2.3 (B), SW2.4 (B), SW3.3 (B), SW3.4 (B), SW4.3 (B), SW4.4 (B), TP3.1, U1.3 (OUT), U2.8 (VCC), U3.20 (AVCC), U3.7 (VCC), U4.19 (V+)
Other:
- moved on the sheet: TP1, TP2, TP3, TP4, TP5, TP6

Commit message: pcb_8
Parts:
- J1: value Barrel_Jack_Switch -> Power_inlet_vertical; Mouser PN 490-PJ-102AH -> (none)
Connections:
- net BTN_DWN: now also R6.2, SW2.3 (B), SW2.4 (B); no longer R6.1, SW2.1 (A), SW2.2 (A)
- net BTN_SEL: now also R7.2, SW3.3 (B), SW3.4 (B); no longer R7.1, SW3.1 (A), SW3.2 (A)
- net BTN_UP: now also R8.2, SW4.3 (B), SW4.4 (B); no longer R8.1, SW4.1 (A), SW4.2 (A)
- net GND: now also SW2.1 (A), SW2.2 (A), SW3.1 (A), SW3.2 (A), SW4.1 (A), SW4.2 (A); no longer R6.2, R7.2, R8.2
- net VCC: now also R6.1, R7.1, R8.1; no longer SW2.3 (B), SW2.4 (B), SW3.3 (B), SW3.4 (B), SW4.3 (B), SW4.4 (B)
Other:
- moved on the sheet: R6, R7, R8, SW2, SW3, SW4

Commit message: gerber out 2
Parts:
- U1: Digikey PN (none) -> 497-7255-1-ND; MFG (none) -> STMicroelectronics; MPN (none) -> L7805CDT-TR
Changed lines of the file:
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@@
+      (effects (font (size 1.27 1.27)) hide)
+    )
+    (property "Digikey PN" "497-7255-1-ND" (id 4) (at 67.31 195.58 0)
+      (effects (font (size 1.27 1.27)) hide)
+    )
+    (property "MPN" "L7805CDT-TR" (id 5) (at 67.31 195.58 0)
+      (effects (font (size 1.27 1.27)) hide)
+    )
+    (property "MFG" "STMicroelectronics" (id 6) (at 67.31 195.58 0)
       (effects (font (size 1.27 1.27)) hide)
     )
