File: hps_clock/hps_clock.kicad_pcb (KiCad board)
At the start: 2 copper layers, 118 x 118 mm, 4 parts

Commit message: schematic done..?
Parts:
- moved H4 126.0 mm to (215.0, 140.0)
- moved H1 66.6 mm to (85.0, 60.0)
- moved H3 66.6 mm to (85.0, 140.0)
- moved H2 41.4 mm to (215.0, 60.0)
Other:
- board size 118 x 118 mm -> 140 x 90 mm

Commit message: pcb_first_draft
Parts:
- added BT1: Battery_Cell, footprints:BatteryHolder_Keystone_106_1x20mm, F.Cu at (186.5, 127.0)
- added C1: C_0805_0.1uf, footprints:C_0805_2012Metric, F.Cu at (111.8, 127.0)
- added C2: C_0805_1uf, footprints:C_0805_2012Metric, F.Cu at (101.6, 68.6)
- added C3: C_0805_0.1uf, footprints:C_0805_2012Metric, F.Cu at (111.8, 68.6)
- added C4: C_0805_0.1uf, footprints:C_0805_2012Metric, F.Cu at (139.7, 67.3)
- added C5: C_0805_0.1uf, footprints:C_0805_2012Metric, F.Cu at (139.7, 73.7)
- added C6: C_0805_22pf, footprints:C_0805_2012Metric, F.Cu at (139.7, 81.3)
- added C7: C_0805_22pf, footprints:C_0805_2012Metric, F.Cu at (139.7, 86.4)
- added C8: C_0805_0.1uf, footprints:C_0805_2012Metric, F.Cu at (165.1, 66.0)
- added C9: C_0805_10uf, footprints:C_0805_2012Metric, F.Cu at (165.1, 73.7)
- added D1: LED_0805, footprints:LED_0805_2012Metric, F.Cu at (137.2, 132.1)
- added DS1: LED_Display_1001, footprints:Adafruit-1001-0-0-MFG, F.Cu at (198.1, 86.4)
- added J1: Barrel_Jack_Switch, footprints:PJ-102AH, F.Cu at (91.4, 76.2)
- added J2: Conn_01x06, footprints:PinHeader_1x06_P2.54mm_Vertical, F.Cu at (121.9, 125.7)
- added J3: Conn_02x03_Odd_Even, footprints:PinHeader_2x03_P2.54mm_Vertical, F.Cu at (127.0, 68.6)
- added R1: R_0805_2.2K, footprints:R_0805_2012Metric, F.Cu at (137.2, 127.0)
- added R10: R_0805_4.7K, footprints:R_0805_2012Metric, F.Cu at (137.2, 96.5)
- added R11: R_0805_10K, footprints:R_0805_2012Metric, F.Cu at (139.7, 101.6)
- added R12: R_0805_22K, footprints:R_0805_2012Metric, F.Cu at (165.1, 83.8)
- added R2: PhotoconductivePhotocell, footprints:R_LDR_4.9x4.2mm_P2.54mm_Vertical, F.Cu at (142.2, 111.8)
- added R3: R_0805_100K, footprints:R_0805_2012Metric, F.Cu at (144.8, 119.4)
- added R4: R_0805_47, footprints:R_0805_2012Metric, F.Cu at (111.8, 132.1)
- added R5: R_0805_47, footprints:R_0805_2012Metric, F.Cu at (111.8, 137.2)
- added R6: R_0805_10K, footprints:R_0805_2012Metric, F.Cu at (91.4, 104.1)
- added R7: R_0805_10K, footprints:R_0805_2012Metric, F.Cu at (106.7, 104.1)
- added R8: R_0805_10K, footprints:R_0805_2012Metric, F.Cu at (121.9, 104.1)
- added R9: R_0805_4.7K, footprints:R_0805_2012Metric, F.Cu at (138.8, 91.4)
- added SW1: Omron_B3F_SPST, footprints:SW_SPST_Omron_B3FS-100xP, F.Cu at (99.1, 134.6)
- added SW2: Omron_B3F_SPST, footprints:SW_SPST_Omron_B3FS-100xP, F.Cu at (91.4, 94.0)
- added SW3: Omron_B3F_SPST, footprints:SW_SPST_Omron_B3FS-100xP, F.Cu at (106.7, 94.0)
- added SW4: Omron_B3F_SPST, footprints:SW_SPST_Omron_B3FS-100xP, F.Cu at (121.9, 94.0)
- added U1: L7805, footprints:TO-252-2, F.Cu at (106.7, 76.2)
- added U2: DS1307_DIP-8, footprints:DIP-8_W7.62mm, F.Cu at (171.5, 123.2)
- added U3: ATmega328-PU, footprints:DIP-28_W7.62mm, F.Cu at (146.1, 67.3)
- added U4: MAX7219, footprints:DIP-24_W7.62mm, F.Cu at (176.5, 72.4)
- added Y1: Crystal_32768Hz, footprints:Crystal_SMD_2Pin_3.2x1.5mm, F.Cu at (185.4, 137.2)
- added Y2: Crystal_16MHz, footprints:Crystal_SMD_HC49-SD, F.Cu at (165.1, 94.0)
Routing:
- added copper zone on B.Cu, net GND
- added copper zone on F.Cu, net VCC
