File: hps_clock/hps_clock.kicad_pcb (KiCad board)
At the start: 2 copper layers, 140 x 90 mm, 41 parts, among them J1 Barrel_Jack_Switch, J2 Conn_01x06, J3 Conn_02x03_Odd_Even, SW1 Omron_B3F_SPST, SW2 Omron_B3F_SPST, SW3 Omron_B3F_SPST, SW4 Omron_B3F_SPST, U1 L7805, U2 DS1307_DIP-8, U3 ATmega328-PU, U4 MAX7219, Y1 Crystal_32768Hz, Y2 Crystal_16MHz

Commit message: pcb_second_draft
Parts:
- BT1: moved to B.Cu
- moved J1 123.1 mm to (203.6, 127.0), turned to 90 degrees
- moved R4 112.8 mm to (208.3, 73.7)
- moved R5 106.7 mm to (195.6, 71.1)
- moved U1 103.3 mm to (203.6, 111.8), turned to 90 degrees
- moved C2 102.6 mm to (193.5, 114.3), turned to 90 degrees
- moved J2 101.2 mm to (200.7, 62.2)
- moved SW1 101.2 mm to (177.8, 71.1)
- moved Y1 101.1 mm to (94.0, 94.0), turned to -90 degrees
- moved D1 97.3 mm to (210.8, 68.6)
- moved C1 95.8 mm to (193.0, 76.2)
- moved R1 95.3 mm to (208.3, 63.5)
- moved C3 90.1 mm to (193.5, 106.7), turned to 90 degrees
- moved U2 79.7 mm to (97.8, 92.7)
- moved BT1 70.9 mm to (115.8, 121.9), turned to 180 degrees
- moved C7 63.6 mm to (203.2, 88.9)
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Routing:
- removed copper zone on B.Cu, net GND

Commit message: pcb_3
Parts:
- moved D1 54.7 mm to (156.1, 66.3), turned to 90 degrees
- moved R1 52.2 mm to (156.1, 62.8), turned to 90 degrees
- moved C7 43.3 mm to (160.0, 86.4)
- moved C8 43.2 mm to (119.4, 78.7), turned to 90 degrees
- moved R12 42.6 mm to (121.9, 78.7), turned to 90 degrees
- moved C9 39.8 mm to (119.4, 74.9), turned to 90 degrees
- moved U4 39.1 mm to (106.7, 90.2)
- moved Y2 36.4 mm to (154.9, 81.3)
- moved C6 35.9 mm to (149.9, 86.4)
- moved R4 34.1 mm to (174.2, 72.5)
- moved J2 23.2 mm to (177.4, 62.4)
- moved R2 23.0 mm to (144.8, 66.0)
- moved R3 22.9 mm to (147.3, 61.0)
- moved R5 21.4 mm to (174.2, 70.1)
- moved C2 19.0 mm to (204.0, 130.1)
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
Commit message: pcb_4
Parts:
- moved C1 32.1 mm to (205.8, 81.1)
- moved R4 32.1 mm to (205.8, 78.5)
- moved J2 32.1 mm to (209.0, 68.4)
- moved R5 32.1 mm to (205.8, 76.1)
- moved R11 32.0 mm to (159.9, 87.3), turned to 90 degrees
- moved C6 27.9 mm to (176.6, 94.2)
- moved C7 27.9 mm to (186.8, 94.2)
- moved R3 27.7 mm to (174.9, 63.0), turned to 90 degrees
- moved SW1 27.3 mm to (196.9, 70.7)
- moved Y2 27.3 mm to (181.6, 87.2)
- moved C5 27.3 mm to (180.4, 72.0)
- moved R10 27.3 mm to (160.0, 72.0)
- moved U3 27.3 mm to (160.1, 83.4)
- moved D1 27.3 mm to (182.8, 71.9)
- moved R1 27.2 mm to (182.7, 68.3)
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
Commit message: pcb_5
Parts:
- added TP1: TestPoint, footprints:TestPoint_THTPad_D2.0mm_Drill1.0mm, F.Cu at (114.0, 103.2)
- added TP2: TestPoint, footprints:TestPoint_THTPad_D2.0mm_Drill1.0mm, F.Cu at (110.4, 105.7)
- added TP3: TestPoint, footprints:TestPoint_THTPad_D2.0mm_Drill1.0mm, F.Cu at (215.7, 108.9)
- added TP4: TestPoint, footprints:TestPoint_THTPad_D2.0mm_Drill1.0mm, F.Cu at (141.6, 92.3)
- added TP5: TestPoint, footprints:TestPoint_THTPad_D2.0mm_Drill1.0mm, F.Cu at (113.7, 92.3)
- added TP6: TestPoint, footprints:TestPoint_THTPad_D2.0mm_Drill1.0mm, F.Cu at (141.7, 78.4)
- J1: footprint footprints:PJ-102AH -> footprints:Wurth-694106402002
- moved C3 15.7 mm to (211.3, 104.4)
- moved U1 14.6 mm to (207.1, 111.1)
- moved C2 13.1 mm to (208.2, 117.7), turned to 180 degrees
- moved C8 4.32 mm to (126.4, 77.9)
- moved C9 4.32 mm to (126.4, 74.1)
- moved R12 4.32 mm to (128.9, 77.9)
- moved U4 4.32 mm to (113.7, 89.3)
- moved J1 1.94 mm to (212.7, 125.1)
Connections:
- BT1 pad 2: GND -> SDA
- C2 pad 2: GND -> SDA
- C3 pad 1: VCC -> SDA
- C3 pad 2: GND -> SDA
- C4 pad 2: GND -> SDA
- C5 pad 1: VCC -> SDA
- C5 pad 2: GND -> SDA
- C6 pad 1: GND -> SDA
- C7 pad 1: GND -> SDA
- C8 pad 1: VCC -> SDA
- C8 pad 2: GND -> SDA
- C9 pad 1: VCC -> SDA
- C9 pad 2: GND -> SDA
- J1 pad 2: GND -> SDA
- J2 pad 1: GND -> SDA
- J2 pad 2: GND -> SDA
- J3 pad 2: VCC -> SDA
- J3 pad 6: GND -> SDA
- R1 pad 2: GND -> SDA
- R10 pad 1: VCC -> SDA
- R10 pad 2: SCL -> SDA
- R11 pad 1: VCC -> SDA
- R12 pad 1: VCC -> SDA
- R2 pad 1: VCC -> SDA
- R3 pad 2: GND -> SDA
- R6 pad 2: GND -> SDA
- R7 pad 2: GND -> SDA
- R8 pad 2: GND -> SDA
- R9 pad 1: VCC -> SDA
- SW1 pad 1: GND -> SDA
- SW1 pad 2: GND -> SDA
- SW2 pad 3: VCC -> SDA
- SW2 pad 4: VCC -> SDA
- SW3 pad 3: VCC -> SDA
- SW3 pad 4: VCC -> SDA
- SW4 pad 3: VCC -> SDA
- SW4 pad 4: VCC -> SDA
- U1 pad 2: GND -> SDA
- U1 pad 3: VCC -> SDA
- U2 pad 4: GND -> SDA
- U2 pad 6: SCL -> SDA
- U2 pad 8: VCC -> SDA
- U3 pad 14: DISP_LOAD -> SDA
- U3 pad 15: DISP_CLK -> SDA
- U3 pad 16: DISP_DATA -> SDA
- U3 pad 20: VCC -> SDA
- U3 pad 22: GND -> SDA
- U3 pad 28: SCL -> SDA
- U3 pad 7: VCC -> SDA
- U3 pad 8: GND -> SDA
- U4 pad 1: DISP_DATA -> SDA
- U4 pad 12: DISP_LOAD -> SDA
- U4 pad 13: DISP_CLK -> SDA
- U4 pad 19: VCC -> SDA
- U4 pad 4: GND -> SDA
- U4 pad 9: GND -> SDA
Routing:
- added copper zone on F.Cu, net SDA
- removed copper zone on F.Cu, net VCC

Commit message: pcb_6
Parts:
- added TP7: TestPoint, footprints:TestPoint_THTPad_D2.0mm_Drill1.0mm, F.Cu at (105.2, 67.7)
- added TP8: TestPoint, footprints:TestPoint_THTPad_D2.0mm_Drill1.0mm, F.Cu at (189.6, 134.0)
- moved TP6 45.1 mm to (96.6, 80.8), turned to 90 degrees
- moved U2 43.5 mm to (128.4, 65.3)
- moved TP1 43.5 mm to (142.6, 70.6)
- moved TP2 43.5 mm to (139.1, 73.0)
- moved Y1 43.5 mm to (124.6, 66.6)
- moved C9 40.6 mm to (92.3, 96.1), turned to 180 degrees
- moved R12 36.3 mm to (96.1, 93.6), turned to 0 degrees
- moved C8 35.3 mm to (96.1, 96.1), turned to 180 degrees
- moved TP4 33.1 mm to (110.5, 80.9), turned to 90 degrees
- moved U4 20.4 mm to (107.5, 108.8), turned to 180 degrees
- moved TP5 16.8 mm to (110.5, 108.8), turned to 90 degrees
- moved J3 7.18 mm to (186.9, 60.9)
- moved D1 5.78 mm to (182.5, 66.1)
- moved R1 5.53 mm to (182.5, 62.7)
- moved R10 4.80 mm to (160.1, 67.2), turned to -90 degrees
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Connections:
- BT1 pad 2: SDA -> GND
- C2 pad 2: SDA -> GND
- C3 pad 1: SDA -> VCC
- C3 pad 2: SDA -> GND
- C4 pad 2: SDA -> GND
- C5 pad 1: SDA -> VCC
- C5 pad 2: SDA -> GND
- C6 pad 1: SDA -> GND
- C7 pad 1: SDA -> GND
- C8 pad 1: SDA -> VCC
- C8 pad 2: SDA -> GND
- C9 pad 1: SDA -> VCC
- C9 pad 2: SDA -> GND
- J1 pad 2: SDA -> GND
- J2 pad 1: SDA -> GND
- J2 pad 2: SDA -> GND
- J3 pad 2: SDA -> VCC
- J3 pad 6: SDA -> GND
- R1 pad 2: SDA -> GND
- R10 pad 1: SDA -> VCC
- R10 pad 2: SDA -> SCL
- R11 pad 1: SDA -> VCC
- R12 pad 1: SDA -> VCC
- R2 pad 1: SDA -> VCC
- R3 pad 2: SDA -> GND
- R6 pad 2: SDA -> GND
- R7 pad 2: SDA -> GND
- R8 pad 2: SDA -> GND
- R9 pad 1: SDA -> VCC
- SW1 pad 1: SDA -> GND
- SW1 pad 2: SDA -> GND
- SW2 pad 3: SDA -> VCC
- SW2 pad 4: SDA -> VCC
- SW3 pad 3: SDA -> VCC
- SW3 pad 4: SDA -> VCC
- SW4 pad 3: SDA -> VCC
- SW4 pad 4: SDA -> VCC
- TP1 pad 1: SDA -> SCL
- TP3 pad 1: SDA -> VCC
- TP4 pad 1: SDA -> DISP_LOAD
- TP5 pad 1: SDA -> DISP_DATA
- TP6 pad 1: SDA -> DISP_CLK
- U1 pad 2: SDA -> GND
- U1 pad 3: SDA -> VCC
- U2 pad 4: SDA -> GND
- U2 pad 6: SDA -> SCL
- U2 pad 8: SDA -> VCC
- U3 pad 14: SDA -> DISP_LOAD
- U3 pad 15: SDA -> DISP_CLK
- U3 pad 16: SDA -> DISP_DATA
- U3 pad 20: SDA -> VCC
- U3 pad 22: SDA -> GND
- U3 pad 28: SDA -> SCL
- U3 pad 7: SDA -> VCC
- U3 pad 8: SDA -> GND
- U4 pad 1: SDA -> DISP_DATA
- U4 pad 12: SDA -> DISP_LOAD
- U4 pad 13: SDA -> DISP_CLK
- U4 pad 19: SDA -> VCC
- U4 pad 4: SDA -> GND
- U4 pad 9: SDA -> GND
Routing:
- net DISP_DATA: track 0.00 -> 107.3 mm, vias 0 -> 2
- net DISP_LOAD: track 0.00 -> 104.0 mm, vias 0 -> 2
- net DISP_CLK: track 0.00 -> 98.7 mm, vias 0 -> 1
- net Net-(DS1-Pad3): track 0.00 -> 72.4 mm, vias 0 -> 1
- net ~{RESET}: track 0.00 -> 68.6 mm
- net BTN_DWN: track 0.00 -> 66.3 mm, vias 0 -> 1
- net Net-(BT1-Pad1): track 0.00 -> 65.6 mm, vias 0 -> 1
- net Net-(DS1-Pad6): track 0.00 -> 63.8 mm, vias 0 -> 1
- net Net-(DS1-Pad5): track 0.00 -> 61.0 mm, vias 0 -> 1
- net Net-(DS1-Pad7): track 0.00 -> 60.8 mm, vias 0 -> 1
- net Net-(DS1-Pad12): track 0.00 -> 59.6 mm, vias 0 -> 1
- net Net-(DS1-Pad9): track 0.00 -> 59.1 mm, vias 0 -> 1
- net BTN_SEL: track 0.00 -> 57.2 mm, vias 0 -> 3
- net Net-(DS1-Pad13): track 0.00 -> 56.9 mm, vias 0 -> 2
- net Net-(DS1-Pad11): track 0.00 -> 55.6 mm, vias 0 -> 1
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- added copper zone on B.Cu, net GND
- added copper zone on F.Cu, net GND
- added copper zone on F.Cu, net VCC
- removed copper zone on F.Cu, net SDA

Commit message: pcb_7
Routing:
- removed copper zone on F.Cu, net GND
Changed lines of the file:
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@@
   (segment (start 191.971089 76.887911) (end 120.499711 76.887911) (width 0.2032) (layer "B.Cu") (net 51))
   (zone (net 6) (net_name "VCC") (layer "F.Cu") (hatch edge 0.508)
-    (connect_pads (clearance 0.508))
+    (connect_pads (clearance 0.3048))
     (min_thickness 0.3048) (filled_areas_thickness no)
     (fill yes (thermal_gap 0.508) (thermal_bridge_width 0.508))
@@
     )
   )
-  (zone (net 2) (net_name "GND") (layer "F.Cu") (hatch edge 0.508)
-    (connect_pads (clearance 0.508))
-    (min_thickness 0.3048) (filled_areas_thickness no)
-    (fill yes (thermal_gap 0.508) (thermal_bridge_width 0.508))
-    (polygon
-      (pts
-        (xy 76.2 53.6956)
-        (xy 75.819 149.9108)
-        (xy 226.0854 149.9108)
-        (xy 225.9076 53.6956)
-        (xy 76.4032 53.4924)
-      )
-    )
-  )
   (zone locked (net 0) (net_name "") (layers F&B.Cu) (hatch edge 0.508)
     (connect_pads (clearance 0))
@@
   (zone (net 2) (net_name "GND") (layer "B.Cu") (hatch edge 0.508)
     (priority 1)
+    (connect_pads (clearance 0.3048))
+    (min_thickness 0.3048) (filled_areas_thickness no)
+    (fill (thermal_gap 0.508) (thermal_bridge_width 0.508))
+    (polygon
+      (pts
+        (xy 226.7458 53.5178)
+        (xy 227.2284 149.8346)
+        (xy 75.946 149.8346)
+        (xy 76.2762 52.9844)
+      )
+    )
+  )
+  (zone (net 2) (net_name "GND") (layer "B.Cu") (hatch edge 0.508)
     (connect_pads (clearance 0.508))
     (min_thickness 0.3048) (filled_areas_thickness no)
@@
     (polygon
       (pts
-        (xy 226.7458 53.5178)
-        (xy 227.2284 149.8346)
-        (xy 75.946 149.8346)
-        (xy 76.2762 53.0352)
-      )
-    )
+        (xy 76.2 53.6956)
+        (xy 76.581 149.9108)
+        (xy -73.6854 149.9108)
+        (xy -73.5076 53.6956)
+        (xy 75.9968 53.4924)
+      )
+    )

Commit message: pcb_8
Parts:
- J1: value Barrel_Jack_Switch -> Power_inlet_vertical; moved to B.Cu
- moved J1 8.82 mm to (200.0, 125.3)
- moved R7 4.84 mm to (148.2, 127.7), turned to 0 degrees
- moved R8 4.73 mm to (163.4, 127.7), turned to 0 degrees
- moved R6 4.65 mm to (132.7, 127.7), turned to 0 degrees
- moved Y2 1.66 mm to (181.8, 88.9)
Connections:
- R6 pad 1: BTN_DWN -> VCC
- R6 pad 2: GND -> BTN_DWN
- R7 pad 1: BTN_SEL -> VCC
- R7 pad 2: GND -> BTN_SEL
- R8 pad 1: BTN_UP -> VCC
- R8 pad 2: GND -> BTN_UP
- SW2 pad 1: BTN_DWN -> GND
- SW2 pad 2: BTN_DWN -> GND
- SW2 pad 3: VCC -> BTN_DWN
- SW2 pad 4: VCC -> BTN_DWN
- SW3 pad 1: BTN_SEL -> GND
- SW3 pad 2: BTN_SEL -> GND
- SW3 pad 3: VCC -> BTN_SEL
- SW3 pad 4: VCC -> BTN_SEL
- SW4 pad 1: BTN_UP -> GND
- SW4 pad 2: BTN_UP -> GND
- SW4 pad 3: VCC -> BTN_UP
- SW4 pad 4: VCC -> BTN_UP
Routing:
- net VCC: track 34.6 -> 15.1 mm
- net BTN_DWN: track 66.3 -> 71.5 mm
- net BTN_UP: track 52.9 -> 58.0 mm
- net BTN_SEL: track 57.2 -> 61.8 mm
- net GND: track 46.1 -> 49.5 mm, vias 19 -> 22
- net Net-(C2-Pad1): track 10.6 -> 12.2 mm

Commit message: gerber out
Other:
- board text added: "bingle board"
